File: MinthySynth/MinthySynth.sch (KiCad schematic (older format))
At the start: 32 parts, among them J1 Conn_01x06_Female, J2 AudioJack3_Ground, J3 Conn_01x06_Female, SW1 SW_SPDT, SW2 SW_Push_Dual, SW3 SW_Push_Dual, SW4 SW_Push_Dual, SW5 SW_Push_Dual, SW6 SW_Push_Dual, SW7 SW_Push_Dual, U1 ATmega328-PU, X1 GTXO-S14T, Y1 16 Mhz

Commit message: Add files via upload
Parts:
- removed X1: GTXO-S14T, Oscillator:Oscillator_DIP-14, symbol Oscillator:GTXO-S14T
- added J4: Conn_01x03_Female, Connector_PinSocket_2.54mm:PinSocket_1x03_P2.54mm_Horizontal, symbol Connector:Conn_01x03_Female
- added J5, J6: Conn_01x01_Female, Connector_PinSocket_2.54mm:PinSocket_1x01_P2.54mm_Vertical, symbol Connector:Conn_01x01_Female
- BT1, BT2: footprint (none) -> bateria:Keystone82
- C1: value CP1 -> 100uF; footprint (none) -> Capacitor_THT:CP_Radial_D12.5mm_P7.50mm
- C2: value C -> 100 nF; footprint (none) -> Capacitor_THT:C_Disc_D3.0mm_W1.6mm_P2.50mm
- C3, C4: footprint (none) -> Capacitor_THT:C_Disc_D3.0mm_W1.6mm_P2.50mm
- D1, D2: footprint (none) -> LED_THT:LED_D3.0mm
- J1: footprint (none) -> Connector_PinHeader_2.54mm:PinHeader_1x06_P2.54mm_Vertical
- J2: footprint (none) -> Connector_Audio:Jack5pin
- J3: footprint (none) -> Connector_PinSocket_2.54mm:PinSocket_1x06_P2.54mm_Vertical
- R1, R2, R3, R4, R5: footprint (none) -> Resistor_THT:R_Axial_DIN0204_L3.6mm_D1.6mm_P5.08mm_Horizontal
- R6: footprint OptoDevice:R_LDR_10x8.5mm_P7.6mm_Vertical -> OptoDevice:R_LDR_7x6mm_P5.1mm_Vertical
- RV1, RV2, RV3, RV4, RV5: footprint (none) -> Potentiometer_THT:Potentiometer_Alps_RK09K_Single_Vertical
- SW1: footprint (none) -> Button_Switch_THT:SW_E-Switch_EG2219_DPDT_Angled
- SW2, SW3, SW4, SW5, SW6, SW7: footprint (none) -> Button_Switch_THT:SW_PUSH_6mm_H5mm
- Y1: footprint (none) -> Crystal:Resonator-3Pin_W7.0mm_H2.5mm
Connections:
- net +3V3: now also J4.2 (Pin_2); no longer BT2.2 (-), C2.1, C3.2, D1.1 (K), D2.1 (K), J2.3, J3.5 (Pin_5), J3.6 (Pin_6), R5.1, RV1.1, RV2.1, RV3.1, RV4.1, RV5.1, SW2.1, SW2.3, SW3.1, SW3.3, SW4.1, SW4.3, SW5.2, SW5.4, SW6.1, SW6.3, SW7.1, SW7.3, U1.22 (GND), U1.8 (GND), Y1.2
- net at U1.18 (PB4): now also J5.1 (Pin_1)
- net at U1.19 (PB5): now also J6.1 (Pin_1)
- net 3: no longer names the net of J3.2 (Pin_2), U1.3 (PD1)
- net 3: now also J4.3 (Pin_3)
- new net GND: BT2.2 (-), C2.1, C3.2, D1.1 (K), D2.1 (K), J2.3, J3.5 (Pin_5), J3.6 (Pin_6), J4.1 (Pin_1), R5.1, RV1.1, RV2.1, RV3.1, RV4.1, RV5.1, SW2.1, SW2.3, SW3.1, SW3.3, SW4.1, SW4.3, SW5.2, SW5.4, SW6.1, SW6.3, SW7.1, SW7.3, U1.22 (GND), U1.8 (GND), Y1.2
- no-connect marks 2 -> 0
Other:
- moved on the sheet: BT1, BT2, C1, C2, C3, C4, D1, D2, J1, J2, J3, R1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
